File: KiCad files/Custom1/TVZ_kuglica_8/TVZ_kuglica.kicad_pcb (KiCad board)
At the start: 2 copper layers, 70 x 80 mm, 34 parts, among them SW1 SW_SPDT

Commit message: to-do
Other:
- net class Default removed

Commit message: footprint
Parts:
- BT1: value 2xAAA -> Battery; footprint TVZ_kuglica:BAT-2xAAA-horizontalni_padovi -> TVZ_kuglica:2xAAA-422-SMT
- moved BT1 53.9 mm to (190.8, 96.2), turned to 180 degrees
Connections:
- BT1 pad 2: GND -> unconnected-(BT1-Pad2)
- SW1 pad 3: Net-(SW1-Pad3) -> unconnected-(SW1-Pad3)
Routing:
- net unconnected-(BT1-Pad2): vias 0 -> 1
- net GND: vias 25 -> 24

Commit message: battery
Parts:
- moved BT1 53.9 mm to (137.0, 100.0)
- moved R3 20.1 mm to (123.0, 78.0)
- moved R6 9.50 mm to (123.5, 130.0)
- moved D8 7.62 mm to (164.2, 105.0)
- moved R7 7.62 mm to (160.5, 105.0)
- moved D3 2.30 mm to (146.0, 76.5)
- moved D7 0.35 mm to (137.0, 130.0)
Routing:
- net Net-(R1-Pad1): track 210.0 -> 0.00 mm
- net VCC: track 41.6 -> 0.00 mm
- net Net-(D11-Pad1): track 19.9 -> 0.00 mm, vias 1 -> 0
- net unconnected-(BT1-Pad2): track 0.00 -> 11.0 mm, vias 1 -> 0
- net Net-(D4-Pad1): track 8.45 -> 0.00 mm, vias 1 -> 0
- net Net-(D8-Pad1): track 3.02 -> 0.00 mm, vias 1 -> 0
- net Net-(D7-Pad1): track 3.02 -> 0.00 mm, vias 1 -> 0
- net Net-(D5-Pad1): track 3.02 -> 0.00 mm, vias 1 -> 0
- net Net-(D3-Pad1): track 3.02 -> 0.00 mm, vias 1 -> 0
- net Net-(D2-Pad1): track 3.02 -> 0.00 mm, vias 1 -> 0
- net Net-(D1-Pad1): track 3.02 -> 0.00 mm, vias 1 -> 0
- net GND: vias 24 -> 0

Commit message: done
Parts:
- removed D1, D4: RGB, TVZ_kuglica:LED-0807
- removed R1, R4: 2k, Resistor_SMD:R_0603_1608Metric
- moved R8 29.6 mm to (122.7, 94.0), turned to 0 degrees
- moved R3 28.5 mm to (151.5, 76.5), turned to 180 degrees
- moved R6 6.50 mm to (123.5, 123.5)
- turned D3 to 180 degrees
Routing:
- net Net-(R2-Pad1): track 0.00 -> 187.8 mm
- net VCC: track 0.00 -> 65.7 mm
- net Net-(D7-Pad1): track 0.00 -> 17.9 mm, vias 0 -> 1
- net Net-(D11-Pad1): track 0.00 -> 16.1 mm, vias 0 -> 1
- net Net-(D3-Pad1): track 0.00 -> 4.77 mm, vias 0 -> 1
- net Net-(D8-Pad1): track 0.00 -> 3.02 mm, vias 0 -> 1
- net Net-(D5-Pad1): track 0.00 -> 3.02 mm, vias 0 -> 1
- net Net-(D2-Pad1): track 0.00 -> 3.02 mm, vias 0 -> 1
- net unconnected-(BT1-Pad2): track 11.0 -> 13.7 mm
- net GND: vias 0 -> 8
