File: KiCad files/Custom1/TVZ_kuglica_8/TVZ_kuglica.kicad_sch (KiCad schematic)
At the start: 18 parts, among them SW1 SW_SPDT

Commit message: footprint
Parts:
- removed BT1: 2xAAA, TVZ_kuglica:BAT-2xAAA-horizontalni_padovi, symbol Device:Battery_Cell
- added BT1: Battery, TVZ_kuglica:2xAAA-422-SMT, symbol Symbols:Battery
Connections:
- net GND: now also BT1.3 (-)
- net VCC: now also BT1.1 (+)
Changed lines of the file:
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@@
-    (stroke (width 0) (type default) (color 0 0 0 0))
-  )
-  (wire (pts (xy 87.63 67.945) (xy 78.74 67.945))
     (stroke (width 0) (type default) (color 0 0 0 0))
   )
@@
     (stroke (width 0) (type default) (color 0 0 0 0))
   )
+  (wire (pts (xy 78.74 73.66) (xy 78.74 67.945))
+    (stroke (width 0) (type default) (color 0 0 0 0))
+  )
   (wire (pts (xy 203.2 74.295) (xy 203.2 78.74))
     (stroke (width 0) (type default) (color 0 0 0 0))
@@
     (stroke (width 0) (type default) (color 0 0 0 0))
   )
+  (wire (pts (xy 78.74 67.945) (xy 87.63 67.945))
+    (stroke (width 0) (type default) (color 0 0 0 0))
+  )
   (wire (pts (xy 101.6 83.82) (xy 101.6 89.535))
     (stroke (width 0) (type default) (color 0 0 0 0))
@@
     (stroke (width 0) (type default) (color 0 0 0 0))
   )
-  (wire (pts (xy 78.74 67.945) (xy 78.74 80.01))
-    (stroke (width 0) (type default) (color 0 0 0 0))
-  )
   (wire (pts (xy 101.6 74.295) (xy 101.6 78.74))
     (stroke (width 0) (type default) (color 0 0 0 0))
@@
     (stroke (width 0) (type default) (color 0 0 0 0))
   )
-  (wire (pts (xy 78.74 89.535) (xy 78.74 87.63))
+  (wire (pts (xy 78.74 83.82) (xy 78.74 89.535))
     (stroke (width 0) (type default) (color 0 0 0 0))
   )
   (wire (pts (xy 172.72 69.215) (xy 172.72 65.405))
     (stroke (width 0) (type default) (color 0 0 0 0))
-  )
-  (symbol (lib_id "Device:Battery_Cell") (at 78.74 85.09 0) (unit 1)
-    (in_bom yes) (on_board yes)
-    (property "Reference" "BT1" (id 0) (at 81.7372 82.6516 0)
-      (effects (font (size 1.27 1.27)) (justify left))
-    )
-    (property "Value" "2xAAA" (id 1) (at 81.7372 84.963 0)
-      (effects (font (size 1.27 1.27)) (justify left))
-    )
-    (property "Footprint" "TVZ_kuglica:BAT-2xAAA-horizontalni_padovi" (id 2) (at 78.74 83.566 90)
-      (effects (font (size 1.27 1.27)) hide)
-    )
-    (property "Datasheet" "~" (id 3) (at 78.74 83.566 90)
-      (effects (font (size 1.27 1.27)) hide)
-    )
-    (pin "1")
-    (pin "2")
   )
   (symbol (lib_id "Device:LED_Small") (at 101.6 81.28 270) (unit 1)
@@
     (pin "2")
   )
+  (symbol (lib_id "Symbols:Battery") (at 78.74 78.74 0) (unit 1)
+    (in_bom yes) (on_board yes) (fields_autoplaced)
+    (property "Reference" "BT1" (id 0) (at 81.407 77.4505 0)
+      (effects (font (size 1.27 1.27)) (justify left))
+    )
+    (property "Value" "Battery" (id 1) (at 81.407 80.2256 0)
+      (effects (font (size 1.27 1.27)) (justify left))
+    )
+    (property "Footprint" "TVZ_kuglica:2xAAA-422-SMT" (id 2) (at 78.74 77.216 90)
+      (effects (font (size 1.27 1.27)) hide)
+    )
+    (property "Datasheet" "~" (id 3) (at 78.74 77.216 90)
+      (effects (font (size 1.27 1.27)) hide)
+    )
+    (pin "1")
+    (pin "2")
+    (pin "3")
+  )
   (sheet_instances
     (path "/" (page "1"))
@@
       (reference "#PWR0102") (unit 1) (value "VCC") (footprint "")
     )
-    (path "/00000000-0000-0000-0000-000061694f6d"
-      (reference "BT1") (unit 1) (value "2xAAA") (footprint "TVZ_kuglica:BAT-2xAAA-horizontalni_padovi")
+    (path "/aa59bb5d-d42e-4add-ad71-ccd5a681621d"
+      (reference "BT1") (unit 1) (value "Battery") (footprint "TVZ_kuglica:2xAAA-422-SMT")
     )
     (path "/00000000-0000-0000-0000-0000616966af"

Commit message: done
Parts:
- removed D1, D4: RGB, TVZ_kuglica:LED-0807, symbol Device:LED_Small
- removed R1, R4: 2k, Resistor_SMD:R_0603_1608Metric, symbol Device:R_Small
Changed lines of the file:
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@@
   (junction (at 142.24 89.535) (diameter 0) (color 0 0 0 0)
   )
-  (junction (at 101.6 65.405) (diameter 0) (color 0 0 0 0)
-  )
   (junction (at 111.76 89.535) (diameter 0) (color 0 0 0 0)
   )
@@
   (junction (at 78.74 67.945) (diameter 0) (color 0 0 0 0)
   )
-  (junction (at 101.6 89.535) (diameter 0) (color 0 0 0 0)
-  )
-  (junction (at 132.08 89.535) (diameter 0) (color 0 0 0 0)
-  )
   (junction (at 163.195 89.535) (diameter 0) (color 0 0 0 0)
   )
-  (junction (at 132.08 65.405) (diameter 0) (color 0 0 0 0)
-  )
   (junction (at 163.195 65.405) (diameter 0) (color 0 0 0 0)
   )
   (no_connect (at 97.79 70.485))
-  (wire (pts (xy 121.92 89.535) (xy 132.08 89.535))
+  (wire (pts (xy 121.92 89.535) (xy 142.24 89.535))
     (stroke (width 0) (type default) (color 0 0 0 0))
   )
@@
     (stroke (width 0) (type default) (color 0 0 0 0))
   )
-  (wire (pts (xy 111.76 65.405) (xy 101.6 65.405))
-    (stroke (width 0) (type default) (color 0 0 0 0))
-  )
-  (wire (pts (xy 132.08 83.82) (xy 132.08 89.535))
-    (stroke (width 0) (type default) (color 0 0 0 0))
-  )
-  (wire (pts (xy 132.08 74.295) (xy 132.08 78.74))
+  (wire (pts (xy 97.79 65.405) (xy 111.76 65.405))
     (stroke (width 0) (type default) (color 0 0 0 0))
   )
@@
     (stroke (width 0) (type default) (color 0 0 0 0))
   )
-  (wire (pts (xy 101.6 65.405) (xy 97.79 65.405))
-    (stroke (width 0) (type default) (color 0 0 0 0))
-  )
   (wire (pts (xy 142.24 89.535) (xy 163.195 89.535))
     (stroke (width 0) (type default) (color 0 0 0 0))
@@
     (stroke (width 0) (type default) (color 0 0 0 0))
   )
-  (wire (pts (xy 101.6 69.215) (xy 101.6 65.405))
-    (stroke (width 0) (type default) (color 0 0 0 0))
-  )
   (wire (pts (xy 142.24 83.82) (xy 142.24 89.535))
     (stroke (width 0) (type default) (color 0 0 0 0))
@@
     (stroke (width 0) (type default) (color 0 0 0 0))
   )
-  (wire (pts (xy 101.6 83.82) (xy 101.6 89.535))
-    (stroke (width 0) (type default) (color 0 0 0 0))
-  )
-  (wire (pts (xy 101.6 89.535) (xy 111.76 89.535))
-    (stroke (width 0) (type default) (color 0 0 0 0))
-  )
-  (wire (pts (xy 132.08 69.215) (xy 132.08 65.405))
+  (wire (pts (xy 78.74 89.535) (xy 111.76 89.535))
     (stroke (width 0) (type default) (color 0 0 0 0))
   )
@@
     (stroke (width 0) (type default) (color 0 0 0 0))
   )
-  (wire (pts (xy 78.74 89.535) (xy 101.6 89.535))
-    (stroke (width 0) (type default) (color 0 0 0 0))
-  )
   (wire (pts (xy 78.74 66.675) (xy 78.74 67.945))
     (stroke (width 0) (type default) (color 0 0 0 0))
@@
     (stroke (width 0) (type default) (color 0 0 0 0))
   )
-  (wire (pts (xy 142.24 65.405) (xy 132.08 65.405))
-    (stroke (width 0) (type default) (color 0 0 0 0))
-  )
   (wire (pts (xy 111.76 89.535) (xy 121.92 89.535))
     (stroke (width 0) (type default) (color 0 0 0 0))
@@
     (stroke (width 0) (type default) (color 0 0 0 0))
   )
-  (wire (pts (xy 101.6 74.295) (xy 101.6 78.74))
-    (stroke (width 0) (type default) (color 0 0 0 0))
-  )
-  (wire (pts (xy 132.08 65.405) (xy 121.92 65.405))
-    (stroke (width 0) (type default) (color 0 0 0 0))
-  )
-  (wire (pts (xy 132.08 89.535) (xy 142.24 89.535))
+  (wire (pts (xy 121.92 65.405) (xy 142.24 65.405))
     (stroke (width 0) (type default) (color 0 0 0 0))
   )
@@
     (stroke (width 0) (type default) (color 0 0 0 0))
   )
-  (symbol (lib_id "Device:LED_Small") (at 101.6 81.28 270) (unit 1)
-    (in_bom yes) (on_board yes)
-    (property "Reference" "D1" (id 0) (at 104.0892 80.1116 90)
-      (effects (font (size 1.27 1.27)) (justify left))
-    )
-    (property "Value" "RGB" (id 1) (at 104.0892 82.423 90)
-      (effects (font (size 1.27 1.27)) (justify left))
-    )
-    (property "Footprint" "TVZ_kuglica:LED-0807" (id 2) (at 101.6 81.28 90)
-      (effects (font (size 1.27 1.27)) hide)
-    )
-    (property "Datasheet" "~" (id 3) (at 101.6 81.28 90)
-      (effects (font (size 1.27 1.27)) hide)
-    )
-    (pin "1")
-    (pin "2")
-  )
   (symbol (lib_id "Device:LED_Small") (at 111.76 81.28 270) (unit 1)
     (in_bom yes) (on_board yes)
@@
     )
     (property "Datasheet" "~" (id 3) (at 121.92 81.28 90)
-      (effects (font (size 1.27 1.27)) hide)
-    )
-    (pin "1")
-    (pin "2")
-  )
-  (symbol (lib_id "Device:LED_Small") (at 132.08 81.28 270) (unit 1)
-    (in_bom yes) (on_board yes)
-    (property "Reference" "D4" (id 0) (at 134.5692 80.1116 90)
-      (effects (font (size 1.27 1.27)) (justify left))
-    )
-    (property "Value" "RGB" (id 1) (at 134.5692 82.423 90)
-      (effects (font (size 1.27 1.27)) (justify left))
-    )
-    (property "Footprint" "TVZ_kuglica:LED-0807" (id 2) (at 132.08 81.28 90)
-      (effects (font (size 1.27 1.27)) hide)
-    )
-    (property "Datasheet" "~" (id 3) (at 132.08 81.28 90)
       (effects (font (size 1.27 1.27)) hide)
     )
@@
     (pin "1")
   )
-  (symbol (lib_id "Device:R_Small") (at 101.6 71.755 0) (unit 1)
-    (in_bom yes) (on_board yes)
-    (property "Reference" "R1" (id 0) (at 103.0986 70.7898 0)
-      (effects (font (size 1.27 1.27)) (justify left))
-    )
-    (property "Value" "2k" (id 1) (at 101.6 72.39 90)
-      (effects (font (size 0.9906 0.9906)) (justify left))
-    )
-    (property "Footprint" "Resistor_SMD:R_0603_1608Metric" (id 2) (at 101.6 71.755 0)
-      (effects (font (size 1.27 1.27)) hide)
-    )
-    (property "Datasheet" "~" (id 3) (at 101.6 71.755 0)
-      (effects (font (size 1.27 1.27)) hide)
-    )
-    (pin "1")
-    (pin "2")
-  )
   (symbol (lib_id "Device:R_Small") (at 111.76 71.755 0) (unit 1)
     (in_bom yes) (on_board yes)
@@
     )
     (property "Datasheet" "~" (id 3) (at 121.92 71.755 0)
-      (effects (font (size 1.27 1.27)) hide)
-    )
-    (pin "1")
-    (pin "2")
-  )
-  (symbol (lib_id "Device:R_Small") (at 132.08 71.755 0) (unit 1)
-    (in_bom yes) (on_board yes)
-    (property "Reference" "R4" (id 0) (at 133.5786 70.7898 0)
-      (effects (font (size 1.27 1.27)) (justify left))
-    )
-    (property "Value" "2k" (id 1) (at 132.08 72.39 90)
-      (effects (font (size 0.9906 0.9906)) (justify left))
-    )
-    (property "Footprint" "Resistor_SMD:R_0603_1608Metric" (id 2) (at 132.08 71.755 0)
-      (effects (font (size 1.27 1.27)) hide)
-    )
-    (property "Datasheet" "~" (id 3) (at 132.08 71.755 0)
       (effects (font (size 1.27 1.27)) hide)
     )
@@
       (reference "BT1") (unit 1) (value "Battery") (footprint "TVZ_kuglica:2xAAA-422-SMT")
     )
-    (path "/00000000-0000-0000-0000-0000616966af"
-      (reference "D1") (unit 1) (value "RGB") (footprint "TVZ_kuglica:LED-0807")
-    )
     (path "/00000000-0000-0000-0000-000061697720"
       (reference "D2") (unit 1) (value "RGB") (footprint "TVZ_kuglica:LED-0807")
@@
       (reference "D3") (unit 1) (value "RGB") (footprint "TVZ_kuglica:LED-0807")
     )
-    (path "/00000000-0000-0000-0000-00006169a5b5"
-      (reference "D4") (unit 1) (value "RGB") (footprint "TVZ_kuglica:LED-0807")
-    )
     (path "/00000000-0000-0000-0000-00006169d1a0"
       (reference "D5") (unit 1) (value "RGB") (footprint "TVZ_kuglica:LED-0807")
@@
       (reference "D11") (unit 1) (value "RGB") (footprint "TVZ_kuglica:LED-0807")
     )
-    (path "/00000000-0000-0000-0000-0000616dc934"
-      (reference "R1") (unit 1) (value "2k") (footprint "Resistor_SMD:R_0603_1608Metric")
-    )
     (path "/00000000-0000-0000-0000-0000616ddade"
       (reference "R2") (unit 1) (value "2k") (footprint "Resistor_SMD:R_0603_1608Metric")
@@
       (reference "R3") (unit 1) (value "2k") (footprint "Resistor_SMD:R_0603_1608Metric")
     )
-    (path "/00000000-0000-0000-0000-0000616dea55"
-      (reference "R4") (unit 1) (value "2k") (footprint "Resistor_SMD:R_0603_1608Metric")
-    )
     (path "/00000000-0000-0000-0000-0000616df2d5"
