File: KiCad files/Custom3/TVZ_kuglica_5/TVZ_kuglica.kicad_pcb (KiCad board)
At the start: 2 copper layers, 70 x 80 mm, 36 parts, among them SW1 SW_SPDT

Commit message: update
Other:
- net class Default removed
